File: self-balancing/native/clock-reset.kicad_sch (KiCad schematic)
At the start: 9 parts, among them U12 TLV803EA29DBZR, X1 8MHz / CL12pF

Commit message: added library and differential rules
Parts:
- C15: footprint Capacitor_SMD:C_0603_1608Metric -> H743_Board:C15_C_0603_1608Metric
- C34: footprint Capacitor_SMD:C_0603_1608Metric -> H743_Board:C34_C_0603_1608Metric
- C35: footprint Capacitor_SMD:C_0603_1608Metric -> H743_Board:C35_C_0603_1608Metric
- C38: footprint Capacitor_SMD:C_0603_1608Metric -> H743_Board:C38_C_0603_1608Metric
- R3: footprint Resistor_SMD:R_0603_1608Metric -> H743_Board:R3_R_0603_1608Metric
- R4: footprint Resistor_SMD:R_0603_1608Metric -> H743_Board:R4_R_0603_1608Metric
- R58: footprint Resistor_SMD:R_0603_1608Metric -> H743_Board:R58_R_0603_1608Metric
- U12: footprint Package_TO_SOT_SMD:SOT-23 -> H743_Board:U12_SOT-23
