File: self-balancing/native/controller.kicad_sch (KiCad schematic)
At the start: 13 parts, among them U1 STM32H743VIT6

Commit message: added library and differential rules
Parts:
- C10: footprint Capacitor_SMD:C_0603_1608Metric -> H743_Board:C10_C_0603_1608Metric
- C11: footprint Capacitor_SMD:C_0603_1608Metric -> H743_Board:C11_C_0603_1608Metric
- C25: footprint Capacitor_SMD:C_0603_1608Metric -> H743_Board:C25_C_0603_1608Metric
- C26: footprint Capacitor_SMD:C_0603_1608Metric -> H743_Board:C26_C_0603_1608Metric
- C3: footprint Capacitor_SMD:C_0603_1608Metric -> H743_Board:C3_C_0603_1608Metric
- C36: footprint Capacitor_SMD:C_0603_1608Metric -> H743_Board:C36_C_0603_1608Metric
- C37: footprint Capacitor_SMD:C_0603_1608Metric -> H743_Board:C37_C_0603_1608Metric
- C6: footprint Capacitor_SMD:C_0603_1608Metric -> H743_Board:C6_C_0603_1608Metric
- C7: footprint Capacitor_SMD:C_0603_1608Metric -> H743_Board:C7_C_0603_1608Metric
- C8: footprint Capacitor_SMD:C_0603_1608Metric -> H743_Board:C8_C_0603_1608Metric
- C9: footprint Capacitor_SMD:C_0603_1608Metric -> H743_Board:C9_C_0603_1608Metric
- R1: footprint Resistor_SMD:R_0603_1608Metric -> H743_Board:R1_R_0603_1608Metric
- U1: footprint Package_QFP:LQFP-100_14x14mm_P0.5mm -> H743_Board:U1_LQFP-100_14x14mm_P0.5mm
Connections:
- net USB_DM_MCU renamed USB_MCU_N
- net USB_DP_MCU renamed USB_MCU_P
