File: self-balancing/native/peripherals.kicad_sch (KiCad schematic)
At the start: 15 parts, among them U10 SN74LVC2G17DBVR, U3 ICM-42688-P

Commit message: added library and differential rules
Parts:
- C12: footprint Capacitor_SMD:C_0603_1608Metric -> H743_Board:C12_C_0603_1608Metric
- C13: footprint Capacitor_SMD:C_0603_1608Metric -> H743_Board:C13_C_0603_1608Metric
- C14: footprint Capacitor_SMD:C_0603_1608Metric -> H743_Board:C14_C_0603_1608Metric
- C31: footprint Capacitor_SMD:C_0603_1608Metric -> H743_Board:C31_C_0603_1608Metric
- R10: footprint Resistor_SMD:R_0603_1608Metric -> H743_Board:R10_R_0603_1608Metric
- R13: footprint Resistor_SMD:R_0603_1608Metric -> H743_Board:R13_R_0603_1608Metric
- R2: footprint Resistor_SMD:R_0603_1608Metric -> H743_Board:R2_R_0603_1608Metric
- R48: footprint Resistor_SMD:R_0603_1608Metric -> H743_Board:R48_R_0603_1608Metric
- R49: footprint Resistor_SMD:R_0603_1608Metric -> H743_Board:R49_R_0603_1608Metric
- R50: footprint Resistor_SMD:R_0603_1608Metric -> H743_Board:R50_R_0603_1608Metric
- R51: footprint Resistor_SMD:R_0603_1608Metric -> H743_Board:R51_R_0603_1608Metric
- R52: footprint Resistor_SMD:R_0603_1608Metric -> H743_Board:R52_R_0603_1608Metric
- R9: footprint Resistor_SMD:R_0603_1608Metric -> H743_Board:R9_R_0603_1608Metric
- U10: footprint Package_TO_SOT_SMD:SOT-23-6 -> H743_Board:U10_SOT-23-6
- U3: footprint Package_LGA:LGA-14_3x2.5mm_P0.5mm_LayoutBorder3x4y -> H743_Board:U3_LGA-14_3x2.5mm_P0.5mm_LayoutBorder3x4y
