File: self-balancing/native/power.kicad_sch (KiCad schematic)
At the start: 31 parts, among them J2 TYPE-C-31-M-12, Q1 2N7002, Q2 DMN2310UW-7, U13 TPS2116DRLR, U2 TPS62162DSGR / 3.3V, U4 USBLC6-2SC6, U6 TPS22918DBVR, U8 TPS3700DDCR

Commit message: added library and differential rules
Parts:
- C1: footprint Capacitor_SMD:C_0805_2012Metric -> H743_Board:C1_C_0805_2012Metric
- C16: footprint Capacitor_SMD:C_0603_1608Metric -> H743_Board:C16_C_0603_1608Metric
- C2: footprint Capacitor_SMD:C_1206_3216Metric -> H743_Board:C2_C_1206_3216Metric
- C24: footprint Capacitor_SMD:C_0603_1608Metric -> H743_Board:C24_C_0603_1608Metric
- C29: footprint Capacitor_SMD:C_0603_1608Metric -> H743_Board:C29_C_0603_1608Metric
- C39: footprint Capacitor_SMD:C_0603_1608Metric -> H743_Board:C39_C_0603_1608Metric
- C4: footprint Capacitor_SMD:C_0603_1608Metric -> H743_Board:C4_C_0603_1608Metric
- C40: footprint Capacitor_SMD:C_0603_1608Metric -> H743_Board:C40_C_0603_1608Metric
- C41: footprint Capacitor_SMD:C_0805_2012Metric -> H743_Board:C41_C_0805_2012Metric
- C5: footprint Capacitor_SMD:C_0603_1608Metric -> H743_Board:C5_C_0603_1608Metric
- Q1: footprint Package_TO_SOT_SMD:SOT-23 -> H743_Board:Q1_SOT-23
- R11: footprint Resistor_SMD:R_0603_1608Metric -> H743_Board:R11_R_0603_1608Metric
- R12: footprint Resistor_SMD:R_0603_1608Metric -> H743_Board:R12_R_0603_1608Metric
- R42: footprint Resistor_SMD:R_0603_1608Metric -> H743_Board:R42_R_0603_1608Metric
- R43: footprint Resistor_SMD:R_0603_1608Metric -> H743_Board:R43_R_0603_1608Metric
- R44: footprint Resistor_SMD:R_0603_1608Metric -> H743_Board:R44_R_0603_1608Metric
- R45: footprint Resistor_SMD:R_0603_1608Metric -> H743_Board:R45_R_0603_1608Metric
- R46: footprint Resistor_SMD:R_0603_1608Metric -> H743_Board:R46_R_0603_1608Metric
- R5: footprint Resistor_SMD:R_0603_1608Metric -> H743_Board:R5_R_0603_1608Metric
- R6: footprint Resistor_SMD:R_0603_1608Metric -> H743_Board:R6_R_0603_1608Metric
- U13: footprint Package_TO_SOT_SMD:SOT-583-8 -> H743_Board:U13_SOT-583-8
- U4: footprint Package_TO_SOT_SMD:SOT-23-6 -> H743_Board:U4_SOT-23-6
- U6: footprint Package_TO_SOT_SMD:SOT-23-6 -> H743_Board:U6_SOT-23-6
Connections:
- net USB_DM_CONN renamed USB_CONN_N
- net USB_DM_ESD renamed USB_ESD_N
- net USB_DM_MCU renamed USB_MCU_N
- net USB_DP_CONN renamed USB_CONN_P
- net USB_DP_ESD renamed USB_ESD_P
- net USB_DP_MCU renamed USB_MCU_P
