File: self-balancing/native/power.kicad_sch (KiCad schematic)
At the start: 31 parts, among them J2 TYPE-C-31-M-12, Q1 2N7002, Q2 DMN2310UW-7, U13 TPS2116DRLR, U2 TPS62162DSGR / 3.3V, U4 USBLC6-2SC6, U6 TPS22918DBVR, U8 TPS3700DDCR

Commit message: Improve H743 schematic readability with wired functional groups
Other:
- note added: "Fixed 3.3 V buck converter"
- note added: "Power mux: stack / slew-limited USB"
- note added: "Stack 5 V health monitor"
- note added: "USB INPUT / SOURCE SELECTION / 3.3 V POWER"
- note added: "USB presence detector"
- note added: "USB slew and source inhibit"
- note added: "USB source disable is controlled by the MCU. Hardware qualification remains pending. TPS62162 uses fixed-3.3 V option: FB grounded; VOS senses after L1. All values, assigned footprints, component identities, and net names are preserved."
- note added: "USB-C termination and ESD"
- note removed: "Routed six-layer prototype CAD | Hardware validation pending"
- note removed: "STorM32 CONTROLLER R3-S | USB-C / BUCK / SOURCE CONTROL"
- moved on the sheet: C1, C16, C2, C24, C29, C39, C4, C40, C41, C5, D4, J2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
