File: self-balancing/native/side-sockets.kicad_sch (KiCad schematic)
At the start: 3 parts, among them J3 MOTOR / 6-wire, J4 EXT SPI SENSOR, J5 GPS / UART4

Commit message: added library and differential rules
Parts:
- J4: footprint Connector_JST:JST_SH_SM08B-SRSS-TB_1x08-1MP_P1.00mm_Horizontal -> H743_Board:J4_JST_SH_SM08B-SRSS-TB_1x08-1MP_P1.00mm_Horizontal
- J5: footprint Connector_JST:JST_SH_SM04B-SRSS-TB_1x04-1MP_P1.00mm_Horizontal -> H743_Board:J5_JST_SH_SM04B-SRSS-TB_1x04-1MP_P1.00mm_Horizontal
