File: self-balancing/native/storage.kicad_sch (KiCad schematic)
At the start: 9 parts, among them U11 W25N01GVZEIG / 128MiB

Commit message: added library and differential rules
Parts:
- C32: footprint Capacitor_SMD:C_0603_1608Metric -> H743_Board:C32_C_0603_1608Metric
- C33: footprint Capacitor_SMD:C_0603_1608Metric -> H743_Board:C33_C_0603_1608Metric
- R53: footprint Resistor_SMD:R_0603_1608Metric -> H743_Board:R53_R_0603_1608Metric
- R54: footprint Resistor_SMD:R_0603_1608Metric -> H743_Board:R54_R_0603_1608Metric
- R55: footprint Resistor_SMD:R_0603_1608Metric -> H743_Board:R55_R_0603_1608Metric
- R56: footprint Resistor_SMD:R_0603_1608Metric -> H743_Board:R56_R_0603_1608Metric
- R57: footprint Resistor_SMD:R_0603_1608Metric -> H743_Board:R57_R_0603_1608Metric
- U11: footprint Package_SON:WSON-8-1EP_8x6mm_P1.27mm_EP3.4x4.3mm -> H743_Board:U11_WSON-8-1EP_8x6mm_P1.27mm_EP3.4x4.3mm
