File: b-rid/b-rid.kicad_sch (KiCad schematic)
At the start: 60 parts, among them J1 USB-C, J2 1S protected pack + NTC, Q1 2N7002P charge isolation, SW1 POWER slide, U1 ESP32-C3-MINI-1-N4X, U2 MIA-M10Q-00B, U3 BQ24074RGT, U4 TPS63031DSK, U5 USBLC6-2SC6, U6 TMUX1119DCKR

Commit message: B-RID: tidy power routing and add USB pair rules
Scope: b-rid only. KiCad 10.0.6 native checks: 0/0/0/0; eight negative rule regression tests pass. Engineering prototype CAD for review; fabrication and battery connection are not released.
Connections:
- net USB_DM renamed USB_D_N
- net USB_DM_CONN renamed USB_D_CONN_N
- net USB_DP renamed USB_D_P
- net USB_DP_CONN renamed USB_D_CONN_P
Changed lines of the file:
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@@
 		)
 	)
-	(label "USB_DP_CONN"
+	(label "USB_D_CONN_P"
 		(at 95.25 107.95 0)
 		(effects
@@
 		)
 	)
-	(label "USB_DP_CONN"
+	(label "USB_D_CONN_P"
 		(at 95.25 110.49 0)
 		(effects
@@
 		)
 	)
-	(label "USB_DM_CONN"
+	(label "USB_D_CONN_N"
 		(at 95.25 102.87 0)
 		(effects
@@
 		)
 	)
-	(label "USB_DM_CONN"
+	(label "USB_D_CONN_N"
 		(at 95.25 105.41 0)
 		(effects
@@
 		)
 	)
-	(label "USB_DP_CONN"
+	(label "USB_D_CONN_P"
 		(at 144.78 99.06 0)
 		(effects
@@
 		)
 	)
-	(label "USB_DP"
+	(label "USB_D_P"
 		(at 144.78 116.84 0)
 		(effects
@@
 		)
 	)
-	(label "USB_DM_CONN"
+	(label "USB_D_CONN_N"
 		(at 160.02 99.06 0)
 		(effects
@@
 		)
 	)
-	(label "USB_DM"
+	(label "USB_D_N"
 		(at 160.02 116.84 0)
 		(effects
@@
 		)
 	)
-	(label "USB_DP_CONN"
+	(label "USB_D_CONN_P"
 		(at 104.14 160.02 0)
 		(effects
@@
 		)
 	)
-	(label "USB_DM_CONN"
+	(label "USB_D_CONN_N"
 		(at 104.14 162.56 0)
 		(effects
@@
 		)
 	)
-	(label "USB_DM_CONN"
+	(label "USB_D_CONN_N"
 		(at 124.46 162.56 0)
 		(effects
@@
 		)
 	)
-	(label "USB_DP_CONN"
+	(label "USB_D_CONN_P"
 		(at 124.46 160.02 0)
 		(effects
@@
 		)
 	)
-	(label "USB_DM"
+	(label "USB_D_N"
 		(at 629.92 320.04 0)
 		(effects
@@
 		)
 	)
-	(label "USB_DP"
+	(label "USB_D_P"
 		(at 629.92 322.58 0)
 		(effects
