File: f722-heli/hardware/f722-heli.kicad_sch (KiCad schematic)
At the start: 15 parts, among them U1 STM32F722RET6

Commit message: F722: add final routed PCB and paired schematics
Parts:
- R16: value 0.15R / 1% / VCAP ESR -> 0.12R / 1% / VCAP ESR; footprint F722_Heli:R_0603_1608Metric -> F722_Heli:R_Panasonic_ERJ3R_0603; LCSC C45879 -> C4059772; MPN 0603WAF150LT5E -> ERJ3RSFR12V; Manufacturer UNI-ROYAL -> Panasonic; Supplier https://jlcpcb.com/partdetail/46882-0603WAF150LT5E/C45879 -> https://jlcpcb.com/partdetail/PANASONIC-ERJ-3RSFR12V/C40597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
