File: f722-heli/hardware/io-ports.kicad_sch (KiCad schematic)
At the start: 31 parts, among them J10 PORT B / JST GH, J11 PORT C / JST GH, J12 DSM / JST ZH, J2 S1 / GND-VX-S, J3 S2 / GND-VX-S, J4 S3 / GND-VX-S, J5 TAIL / GND-VX-S, J6 ESC / GND-VX-S, J7 RPM / GND-VX-S, J8 SBUS / GND-VX-S, J9 PORT A / JST GH, U12 USBLC6-4SC6 / header clamp, U13 USBLC6-4SC6 / header clamp, U14 TPD4E05U06DQAR / UART ESD, U15 TPD4E05U06DQAR / UART ESD

Commit message: F722: add final routed PCB and paired schematics
Parts:
- J2, J3, J4, J5, J6, J7, J8: footprint F722_Heli:Samtec_HTSW-101-08-L-T-RA_TripleRow -> F722_Heli:Samtec_HTSW-101-08-L-T-RA_TripleRow_OpenEdgeSilk
- R31: footprint F722_Heli:R_0402_1005Metric -> F722_YAGEO:R_0201_0603Metric_YAGEO_AC; LCSC C25092 -> C144830; MPN 0402WGF220JTCE -> AC0201FR-0722RL; Manufacturer UNI-ROYAL (Uniroyal Elec) -> YAGEO; Supplier https://jlcpcb.com/partdetail/25835-0402WGF220JTCE/C25092 -> https://jlcpcb.com/partdetail/YAGEO-AC0201FR0722RL/C144830
- U14: symbol F722_Heli:TPD4E05U06 -> F722_Heli:TPD4E05U06_RoutePads
Connections:
- net PORT_A_RX_EXT: now also U14.10 (NC10)
- net PORT_A_TX_EXT: now also U14.9 (NC9)
- net PORT_B_RX_EXT: now also U14.7 (NC7)
- net PORT_B_TX_EXT: now also U14.6 (NC6)
- no-connect marks 11 -> 7
Other:
- note added: "U14 routing lands: NC10/IO1, NC9/IO2, NC7/IO4, NC6/IO5. External PCB copper is required; active IO pads remain the clamps."

Commit message: WIP: open the adopted native3 layout from the normal F722 project
Parts:
- U15: symbol F722_Heli:TPD4E05U06 -> F722_Heli:TPD4E05U06_RoutePads_NC9_NC10
Connections:
- net ESC_MCU: now also U13.3 (I/O2); no longer U13.1 (I/O1)
- net PORT_C_RX_EXT: now also U15.10 (NC10)
- net PORT_C_TX_EXT: now also U15.9 (NC9)
- net RPM_MCU: now also U13.6 (I/O4); no longer U13.3 (I/O2)
- net SBUS_MCU: now also U13.1 (I/O1); no longer U13.6 (I/O4)
- no-connect marks 7 -> 5
