File: f722-heli/hardware/sensors.kicad_sch (KiCad schematic)
At the start: 17 parts, among them U2 ICM-42688-P, U3 W25N01GVZEIG / 128MiB, U4 DPS368XTSA1 / 0x76

Commit message: F722: add final routed PCB and paired schematics
Parts:
- R5: footprint F722_Heli:R_0402_1005Metric -> F722_Heli:R_0402_1005Metric_R5_ClearPin1Silk

Commit message: WIP: open the adopted native3 layout from the normal F722 project
Parts:
- R7, R8: value 4.7k / 1% -> 2.2k / 1%; LCSC C25900 -> C25879; MPN 0402WGF4701TCE -> 0402WGF2201TCE; Supplier https://jlcpcb.com/partdetail/26643-0402WGF4701TCE/C25900 -> https://jlcpcb.com/partdetail/26622-0402WGF2201TCE/C25879
