File: f722-heli/hardware/usb-clock.kicad_sch (KiCad schematic)
At the start: 22 parts, among them J1 USB4105-GF-A-120, SW1 BOOT / KMT031NGJLHS, Y1 8MHz / CL10pF / TAXM8M4RDBCCT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

Commit message: F722: add final routed PCB and paired schematics
Parts:
- J1: value USB4105-GF-A-120 -> USB4145-03-0170-C; footprint F722_Heli:USB_C_Receptacle_GCT_USB4105-xx-A_16P_TopMnt_Horizontal -> F722_Heli:USB_C_Receptacle_GCT_USB4145-03-0170-C_16P_Vertical; LCSC C5184243 -> C5181332; MPN USB4105-GF-A-120 -> USB4145-03-0170-C; Supplier https://jlcpcb.com/partdetail/5849584-USB4105_GF_A120/C5184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 -> https://jlcpcb.com/partdetail/5839804-USB4145_03_0170C/C518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
