File: nexus-style-fc-power-module/hardware/nexus-style-fc-power-module.kicad_sch (KiCad schematic)
At the start: 30 parts, among them J1 PWR IN, J2 PWR OUT, U14 TPS629210DRLR, U5 TPS62130RGTR, U9 TPS2116DRLR

Commit message: added standalone power module
Other:
- note added: "-> MCU PC0"
- note added: "-> MCU PC1"
- note added: "3V3 MCU BUCK TPS629210 1 A, fed from VSYS (VX or VBUS through Schottky OR)"
- note added: "DSM 3V3 PORT FUSE"
- note added: "FSW = GND: 2.5 MHz, DEF = GND"
- note added: "INPUT J1"
- note added: "OUTPUT J2"
- note added: "S-CONF 27.4k = setting 9: VSET mode, FB/VSET open = 3.3 V, auto PFM"
- note added: "Vout = 0.8 V x (1 + 120k / 22k) = 5.16 V"
- note added: "switches to USB below 1.0 V x (100k + 27k) / 27k = 4.7 V"
- note removed: "3V3 MCU BUCK TPS629210 1 A, fed from VSYS (VX or VBUS through Schottky OR) + DSM 3V3 port fuse"
- note removed: "MODULE I/O J1 in | J2 out"
- note removed: "POWER FLAGS"
- moved on the sheet: C21, C22, C23, C24, C25, C26, C27, C28, C29, C30, D4, D5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

Commit message: added usbc
Parts:
- added F1: 0.5A PTC, NexusFC:F0805, symbol NexusFC:SMD0805P050TF
- added J6: USB-C vertical, NexusFC:USB-C-SMD_TYPE-C-31-D-06, symbol NexusFC:TYPE-C-31-D-06
- added R20, R21: 5.1k, Resistor_SMD:R_0402_1005Metric, symbol Device:R
- added U7: USBLC6-2SC6, NexusFC:SOT-23-6_L2.9-W1.6-P0.95-LS2.8-BL, symbol NexusFC:USBLC6-2SC6
- J1: footprint Connector_PinHeader_2.54mm:PinHeader_1x04_P2.54mm_Vertical -> Connector_PinHeader_2.54mm:PinHeader_1x02_P2.54mm_Vertical; symbol Connector_Generic:Conn_01x04 -> Connector_Generic:Conn_01x02
- J2: footprint Connector_PinHeader_2.54mm:PinHeader_1x08_P2.54mm_Vertical -> Connector_PinHeader_2.54mm:PinHeader_1x10_P2.54mm_Vertical; symbol Connector_Generic:Conn_01x08 -> Connector_Generic:Conn_01x10
Connections:
- net 5V_SENSE: now also J2.7 (Pin_7); no longer J2.8 (Pin_8)
- net GND: now also J2.8 (Pin_8), J6.A1 (GND), J6.A12 (GND), J6.B1 (GND), J6.B12 (GND), J6.EP, R20.2, R21.2, U7.2; no longer J1.4 (Pin_4), J2.6 (Pin_6)
- net VBUS: now also F1.2, U7.5; no longer J1.3 (Pin_3)
- net VX_SENSE: now also J2.6 (Pin_6); no longer J2.7 (Pin_7)
- new net CC1: J6.A5 (CC1), R20.1
- new net CC2: J6.B5 (CC2), R21.1
- new net USB_DM: J2.9 (Pin_9), J6.A7 (DN1), J6.B7 (DN2), U7.1, U7.6
- new net USB_DP: J2.10 (Pin_10), J6.A6 (DP1), J6.B6 (DP2), U7.3, U7.4
- new net VBUS_C: F1.1, J6.A4 (VBUS), J6.A9 (VBUS), J6.B4 (VBUS), J6.B9 (VBUS)
- no-connect marks 4 -> 6
Other:
- note added: "SBU1 / SBU2 not used; Rd 5.1k on each CC = 5 V sink (UFP)"
- note added: "USB-C (VBUS PTC, Rd 5.1k on CC, USBLC6 ESD on D+ / D-)"
