File: nexus-style-fc/hardware/nexus-style-fc.kicad_sch (KiCad schematic)
At the start: 88 parts, among them J1 Header child board, J2 DSM (UART1), J3 A-CRSF (UART4), J4 C (UART3), J5 B (UART6), J6 USB-C vertical, SW1 BOOT, U1 STM32F722RET6, U10 TPS70933DBVR, U11 SRV05-4, U12 SRV05-4, U13 SRV05-4, U14 TPS629210DRLR, U15 SRV05-4, U2 ICM-42688-P, U3 DPS368XTSA1, U4 W25N01GVZEIG, U5 TPS62130RGTR, U7 USBLC6-2SC6, U9 TPS2116DRLR, Y1 8MHz 20pF

Commit message: WIP: connect Nexus schematic units and isolate U10 EN; preserve 32-error route checkpoint
Connections:
- net VSYS: no longer U10.3 (EN)
- no-connect marks 25 -> 26
Other:
- note added: "01 VX INPUT / 5 V BUCK"
- note added: "02 5 V SOURCE PRIORITY"
- note added: "03 VSYS / MCU 3.3 V"
- note added: "04 LOW-NOISE SENSOR SUPPLY"
- note added: "05 VOLTAGE MONITORING / POWER FLAGS"
- note added: "06 STM32F722 CORE"
- note added: "07 CLOCK / BOOT / DEBUG"
- note added: "08 MCU DECOUPLING"
- note added: "09 SPI1 INERTIAL SENSOR"
- note added: "10 I2C1 PRESSURE SENSOR"
- note added: "11 USB-C / PROTECTION"
- note added: "12 RECEIVER INTERFACES"
- note added: "13 SERVO HEADER / SIGNAL CLAMPS"
- note added: "14 SPI2 BLACKBOX"
- note added: "15 STATUS INDICATION"
- note added: "5V_BUCK is preferred; USB VBUS supplies 5V when the buck is absent"
- note added: "8 MHz HSE; BOOT selects DFU. SWD pads are for bring-up and debug."
- note added: "A = UART4 (CRSF); B = UART6; C = UART3; DSM = UART1"
- note added: "ADC input dividers: VX_SENSE -> U1.9; 5V_SENSE -> U1.10"
- note added: "C1-4: VDD; C5: bulk; C6-7: VDDA; C8: VBAT; C9: VCAP"
- note added: "DPS368: address 0x76; CSB high selects I2C; R6 / R7 pull up SCL / SDA"
- note added: "Do not tie EN to VSYS. Pin 4 is also intentionally unconnected."
- note added: "ICM-42688-P: IMU_CS / SPI1; IMU_INT -> U1.50; powered by 3V3_SENS"
- note added: "J1 mates with the separate header board; VX and GND enter at pins 1 / 2"
- note added: "NEXUS-STYLE FLIGHT CONTROLLER | FUNCTIONAL SCHEMATIC"
- note added: "PC14 / PC15 sink only: active low, about 1.3 mA. Blue = 5 V bus present."
- note added: "Read left to right: POWER / MCU + SENSORS / INTERFACES. Matching global labels connect across panels."
- note added: "Rotorflight RDMS-NEXUS_F7 pin map; named interfaces continue in panels 09-15"
- note added: "SPI1: IMU | SPI2: blackbox | I2C1: barometer"
- note added: "UNFINISHED PCB CHECKPOINT - NOT RELEASED FOR FABRICATION. X = intentionally unconnected pin."
- note added: "USB 2.0 device; CC1 / CC2 Rd = 5.1k; F1 protects VBUS"
- note added: "VSYS -> U10 -> 3V3_SENS. EN pin 3 intentionally floating (internal pull-up)."
- note added: "VX -> U5 / L1 -> 5V_BUCK; feedback R11 / R12 sets about 5.16 V"
- note added: "VX / VBUS diode-OR -> VSYS -> U14 / L2 -> 3V3; F2 limits the DSM port"
- note added: "W25N01GV 128 MB; /CS, /WP and /HOLD pull-ups; EP intentionally floating"
- note removed: "BLACKBOX W25N01GV 128MB (SPI2)"
- note removed: "LEDs (PC14/PC15 sink only, <=3 mA)"
- note removed: "MCU STM32F722RET6 (Rotorflight RDMS-NEXUS_F7 pinout)"
- note removed: "POWER FLAGS"
- note removed: "POWER VX TVS | 5V buck + USB priority mux | VSYS -> 3V3 MCU buck | DSM 3V3 buck | ADC sense"
- note removed: "RECEIVER PORTS A-CRSF UART4 | B UART6 | C UART3 | DSM UART1 + ESD"
- note removed: "SENSORS ICM-42688-P (SPI1) DPS368 (I2C1 0x76) 3V3_SENS LDO"
- note removed: "SERVO HEADER CHILD BOARD JOINT + clamps"
- note removed: "USB-C (PTC + ESD, Rd 5.1k)"
- moved on the sheet: C1, C10, C11, C12, C13, C14, C15, C16, C17, C18, C19, C2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

Commit message: WIP Nexus: redraw all circuits, apply approved C19 upgrade, checkpoint r43
Native KiCad 10: experimental 29 clearance errors; canonical 627 inherited errors. Both zero opens/parity/ERC and 54 inherited silk warnings. Header retains 11 edge errors. No fabrication release.
Parts:
- C19: value 2.2uF -> 10uF; LCSC C23630 -> C19702
Other:
- note added: "8 MHz HSE with load capacitors; BOOT0 button and pull-down; SWD / reset pads"
- note added: "A: UART4 / CRSF | B: UART6 | C: UART3 | DSM: UART1"
- note added: "ADC divider filters | VX_SENSE -> U1.9; 5V_SENSE -> U1.10"
- note added: "Buck-priority power mux | 5V_BUCK preferred, USB VBUS fallback"
- note added: "CSB = VDDIO; SDO = GND"
- note added: "Crystal case pads -> GND"
- note added: "DPS368 address 0x76: SDO low; CSB high selects I2C; local SCL / SDA pull-ups"
- note added: "Diode-OR supply -> TPS629210 -> MCU rail; fused DSM supply branch"
- note added: "EN and NC are intentionally unconnected. Do not tie EN to VSYS."
- note added: "FSW = GND: 2.5 MHz; DEF = GND"
- note added: "ICM-42688-P; IMU_CS pull-up maintains SPI mode at startup; IMU_INT -> U1.50"
- note added: "J1 connects the separate header board; VX / GND enter at pins 1 / 2"
- note added: "Local 3V3 bypass: C1-4 VDD, C5 bulk, C6-7 VDDA, C8 VBAT; C9 VCAP only"
- note added: "NEXUS-STYLE FLIGHT CONTROLLER | CIRCUIT SCHEMATIC"
- note added: "PC14 / PC15 sink current: active low | Blue indicates 5 V bus power"
- note added: "POWER / COMPUTE + SENSORS / INTERFACES. Named boundaries connect between functional circuits."
- note added: "Press BOOT during reset for DFU"
- note added: "Rotorflight RDMS-NEXUS_F7 pin map; boundary labels connect the functional units"
- note added: "SPI1: inertial sensor | SPI2: blackbox | I2C1: barometer"
- note added: "TPS62130: 3 A, 2.5 MHz | Vout = 0.8 V x (1 + 120k / 22k) = 5.16 V"
- note added: "TPS70933: EN pin 3 intentionally floating, supported by internal pull-up"
- note added: "USB 2.0 device | CC pull-downs: 5.1k | F1: VBUS resettable fuse"
- note added: "VCAP pin 30"
- note added: "VDD pins 19 / 32 / 48 / 64"
- note added: "VDDA pin 13 / VBAT pin 1"
- note added: "W25N01GV 128 MB | /CS, /WP, /HOLD pull-ups | EP intentionally floating"
- note removed: "5V_BUCK is preferred; USB VBUS supplies 5V when the buck is absent"
- note removed: "8 MHz HSE; BOOT selects DFU. SWD pads are for bring-up and debug."
- note removed: "A = UART4 (CRSF); B = UART6; C = UART3; DSM = UART1"
- note removed: "ADC input dividers: VX_SENSE -> U1.9; 5V_SENSE -> U1.10"
- note removed: "C1-4: VDD; C5: bulk; C6-7: VDDA; C8: VBAT; C9: VCAP"
- note removed: "DPS368: address 0x76; CSB high selects I2C; R6 / R7 pull up SCL / SDA"
- note removed: "Do not tie EN to VSYS. Pin 4 is also intentionally unconnected."
- note removed: "ICM-42688-P: IMU_CS / SPI1; IMU_INT -> U1.50; powered by 3V3_SENS"
- note removed: "J1 mates with the separate header board; VX and GND enter at pins 1 / 2"
- note removed: "NEXUS-STYLE FLIGHT CONTROLLER | FUNCTIONAL SCHEMATIC"
- note removed: "PC14 / PC15 sink only: active low, about 1.3 mA. Blue = 5 V bus present."
- note removed: "Read left to right: POWER / MCU + SENSORS / INTERFACES. Matching global labels connect across panels."
- note removed: "Rotorflight RDMS-NEXUS_F7 pin map; named interfaces continue in panels 09-15"
- note removed: "SPI1: IMU | SPI2: blackbox | I2C1: barometer"
- note removed: "USB 2.0 device; CC1 / CC2 Rd = 5.1k; F1 protects VBUS"
- note removed: "VSYS -> U10 -> 3V3_SENS. EN pin 3 intentionally floating (internal pull-up)."
- note removed: "VX -> U5 / L1 -> 5V_BUCK; feedback R11 / R12 sets about 5.16 V"
- note removed: "VX / VBUS diode-OR -> VSYS -> U14 / L2 -> 3V3; F2 limits the DSM port"
- note removed: "W25N01GV 128 MB; /CS, /WP and /HOLD pull-ups; EP intentionally floating"
- moved on the sheet: C1, C10, C11, C12, C13, C14, C15, C16, C17, C18, C19, C2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

Commit message: WIP Nexus r57: 13 clearance errors, contact diagnostics and scoped symbol filters
Preserve canonical copper and unrelated projects. Include native ERC/parity, current schematic PDF/source, off-pad hole and annular-entry proofs. Keep mechanical candidate02 separate and unfinished; no fabrication release.
Parts:
- J1: symbol Connector_Generic:Conn_01x09 -> NexusReviewed:HeaderBoardJoint
- L1, L2: symbol Device:L -> NexusReviewed:PowerInductor
Changed lines of the file:
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@@
 	)
 	(symbol
-		(lib_id "Device:L")
+		(lib_id "NexusReviewed:PowerInductor")
 		(at 184.15 97.79 90)
 		(unit 1)
@@
 	)
 	(symbol
-		(lib_id "Device:L")
+		(lib_id "NexusReviewed:PowerInductor")
 		(at 208.28 322.58 90)
 		(unit 1)
@@
 	)
 	(symbol
-		(lib_id "Connector_Generic:Conn_01x09")
+		(lib_id "NexusReviewed:HeaderBoardJoint")
 		(at 585.47 355.6 180)
 		(unit 1)

Commit message: Consolidate Nexus stage36 into canonical project paths
Preserve matched native sources and manufacturing bytes; use Git history for older project snapshots. Retain revision-bound validation evidence, document open release gates, and guard destructive regeneration.
Parts:
- added C31: 22uF, NexusFC:C_0805_2012Metric_Samsung_CL21_MinLand, symbol Device:C
- C27: value 4.7uF -> 22uF; footprint Capacitor_SMD:C_0603_1608Metric -> NexusFC:C_0805_2012Metric_Samsung_CL21_MinLand; LCSC C69335 -> C602037
- D1: footprint NexusFC:LED0603-RD_GREEN -> NexusFC:LED0603-RD_GREEN__NexusMain_D1
- D2: footprint NexusFC:LED0603-RD_RED -> NexusFC:LED0603-RD_RED__NexusMain_D2
- D3: footprint NexusFC:LED0603-RD_BLUE -> NexusFC:LED0603-RD_BLUE__NexusMain_D3
- J4: footprint NexusFC:CONN-SMD_4P-P1.25_BM04B-GHS-TBT-LF-SN -> NexusFC:CONN-SMD_4P-P1.25_BM04B-GHS-TBT-LF-SN__NexusMain_J4
- J6: footprint NexusFC:USB-C-SMD_TYPE-C-31-D-06 -> NexusFC:USB-C-SMD_TYPE-C-31-D-06__NexusMain_J6
- U10: footprint NexusFC:SOT-23-5_L3.0-W1.7-P0.95-LS2.8-BL -> NexusFC:TPS70933DBVR_TI_DBV0005A
Connections:
- net GND: now also C31.2
- net VSYS: now also C31.1
- net USB_DM renamed USB_DN
Changed lines of the file:
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@@
 			)
 		)
-		(property "Value" "4.7uF"
+		(property "Value" "22uF"
 			(at 102.87 328.93 0)
 			(effects
@@
 			)
 		)
-		(property "Footprint" "Capacitor_SMD:C_0603_1608Metric"
+		(property "Footprint" "NexusFC:C_0805_2012Metric_Samsung_CL21_MinLand"
 			(at 99.06 327.66 0)
 			(effects
@@
 			)
 		)
-		(property "LCSC" "C69335"
+		(property "LCSC" "C602037"
 			(at 99.06 327.66 0)
 			(effects
@@
 			)
 		)
-		(property "Description" "buck in, 25 V"
+		(property "Description" "Main VSYS input bulk; Samsung CL21A226MAYNNNE; 22 uF, 25 V, X5R, +/-20%; JLC/LCSC C602037"
 			(at 99.06 327.66 0)
 			(effects
@@
 		)
 	)
+	(symbol
+		(lib_id "Device:C")
+		(at 71.12 327.66 0)
+		(unit 1)
+		(exclude_from_sim no)
+		(in_bom yes)
+		(on_board yes)
+		(dnp no)
+		(property "Reference" "C31"
+			(at 74.93 326.39 0)
+			(effects
+				(font
+					(size 1.27 1.27)
+				)
+				(justify left)
+			)
+		)
+		(property "Value" "22uF"
+			(at 74.93 328.93 0)
+			(effects
+				(font
+					(size 1.27 1.27)
+				)
+				(justify left)
+			)
+		)
+		(property "Footprint" "NexusFC:C_0805_2012Metric_Samsung_CL21_MinLand"
+			(at 71.12 327.66 0)
+			(effects
+				(font
+					(size 1.27 1.27)
+				)
+				(hide yes)
+			)
+		)
+		(property "Datasheet" ""
+			(at 71.12 327.66 0)
+			(effects
+				(font
+					(size 1.27 1.27)
+				)
+				(hide yes)
+			)
+		)
+		(property "LCSC" "C602037"
+			(at 71.12 327.66 0)
+			(effects
+				(font
+					(size 1.27 1.27)
+				)
+				(hide yes)
+			)
+		)
+		(property "Description" "Main VSYS local parallel input bulk; Samsung CL21A226MAYNNNE; 22 uF, 25 V, X5R, +/-20%; JLC/LCSC C602037"
+			(at 71.12 327.66 0)
+			(effects
+				(font
+					(size 1.27 1.27)
+				)
+				(hide yes)
+			)
+		)
+		(pin "1"
+		)
+		(pin "2"
+		)
+		(instances
+			(project "nexus-style-fc"
+				(path "/b1e839ec-d91a-58d5-9282-f5372deabfab"
+					(reference "C31")
+					(unit 1)
+				)
+			)
+		)
+	)
+	(wire
+		(pts
+			(xy 71.12 323.85)
+			(xy 71.12 317.5)
+		)
+		(stroke
+			(width 0)
+			(type default)
+		)
+	)
+	(junction
+		(at 71.12 317.5)
+		(diameter 0)
+		(color 0 0 0 0)
+	)
+	(wire
+		(pts
+			(xy 71.12 331.47)
+			(xy 71.12 340.36)
+		)
+		(stroke
+			(width 0)
+			(type default)
+		)
+	)
+	(wire
+		(pts
+			(xy 71.12 340.36)
+			(xy 99.06 340.36)
+		)
+		(stroke
+			(width 0)
+			(type default)
+		)
+	)
+	(junction
+		(at 99.06 340.36)
+		(diameter 0)
+		(color 0 0 0 0)
+	)
 	(global_label "VSYS"
 		(shape passive)
@@
 			)
 		)
-		(property "Footprint" "NexusFC:SOT-23-5_L3.0-W1.7-P0.95-LS2.8-BL"
+		(property "Footprint" "NexusFC:TPS70933DBVR_TI_DBV0005A"
 			(at 148.59 422.91 0)
 			(effects
@@
 		)
 	)
-	(global_label "USB_DM"
+	(global_label "USB_DN"
 		(shape passive)
 		(at 450.85 111.76 0)
@@
 			)
 		)
-		(property "Footprint" "NexusFC:USB-C-SMD_TYPE-C-31-D-06"
+		(property "Footprint" "NexusFC:USB-C-SMD_TYPE-C-31-D-06__NexusMain_J6"
 			(at 608.33 96.52 0)
 			(effects
@@
 		)
 	)
-	(global_label "USB_DM"
+	(global_label "USB_DN"
 		(shape passive)
 		(at 590.55 96.52 180)
@@
 		(color 0 0 0 0)
 	)
-	(global_label "USB_DM"
+	(global_label "USB_DN"
 		(shape passive)
 		(at 676.91 101.6 0)
@@
 		)
 	)
-	(global_label "USB_DM"
+	(global_label "USB_DN"
 		(shape passive)
 		(at 763.27 101.6 0)
@@
 			)
 		)
-		(property "Footprint" "NexusFC:CONN-SMD_4P-P1.25_BM04B-GHS-TBT-LF-SN"
+		(property "Footprint" "NexusFC:CONN-SMD_4P-P1.25_BM04B-GHS-TBT-LF-SN__NexusMain_J4"
 			(at 590.55 265.43 90)
 			(effects
@@
 			)
 		)
-		(property "Footprint" "NexusFC:LED0603-RD_GREEN"
+		(property "Footprint" "NexusFC:LED0603-RD_GREEN__NexusMain_D1"
 			(at 612.14 524.51 0)
 			(effects
@@
 			)
 		)
-		(property "Footprint" "NexusFC:LED0603-RD_RED"
+		(property "Footprint" "NexusFC:LED0603-RD_RED__NexusMain_D2"
 			(at 698.5 524.51 0)
 			(effects
@@
 			)
 		)
-		(property "Footprint" "NexusFC:LED0603-RD_BLUE"
+		(property "Footprint" "NexusFC:LED0603-RD_BLUE__NexusMain_D3"
 			(at 786.13 524.51 0)
 			(effects

Commit message: fix(nexus): clean up native fabrication warnings and bind verified exports
Center existing via connections, fix mixed USB connector classification,
move conflicting outline artwork to Fab layers, and synchronize reviewed
symbol/footprint identities. Preserve accepted pads, pinouts and parts.

Regenerate main CAM and record full KiCad 10 ERC/DRC/parity and source/CAM
consistency evidence. Keep remaining factory and bench qualification gates
explicit; this checkpoint is not a fabrication or flight release.
Parts:
- F1: footprint NexusFC:F0805 -> NexusFC:F0805__NexusMain_F1
- F2: footprint NexusFC:F0805 -> NexusFC:F0805__NexusMain_F2
- J2: footprint NexusFC:CONN-SMD_B3B-ZR-SM4-TF -> NexusFC:CONN-SMD_B3B-ZR-SM4-TF__NexusMain_J2
- J3: footprint NexusFC:CONN-SMD_4P-P1.25_BM04B-GHS-TBT-LF-SN -> NexusFC:CONN-SMD_4P-P1.25_BM04B-GHS-TBT-LF-SN__NexusMain_J3
- J5: footprint NexusFC:CONN-SMD_4P-P1.25_BM04B-GHS-TBT-LF-SN -> NexusFC:CONN-SMD_4P-P1.25_BM04B-GHS-TBT-LF-SN__NexusMain_J5
- L2: footprint NexusFC:IND-SMD_L2.0-W1.6 -> NexusFC:IND-SMD_L2.0-W1.6__NexusMain_L2
- R2: footprint Resistor_SMD:R_0402_1005Metric -> NexusFC:R_0402_1005Metric__NexusMain_R2
- R4: footprint Resistor_SMD:R_0402_1005Metric -> NexusFC:R_0402_1005Metric__NexusMain_R4
- Y1: footprint NexusFC:CRYSTAL-SMD_4P-L3.2-W2.5-BL -> NexusFC:CRYSTAL-SMD_4P-L3.2-W2.5-BL__NexusMain_Y1
Changed lines of the file:
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@@
 			)
 		)
-		(property "Footprint" "NexusFC:IND-SMD_L2.0-W1.6"
+		(property "Footprint" "NexusFC:IND-SMD_L2.0-W1.6__NexusMain_L2"
 			(at 208.28 322.58 90)
 			(effects
@@
 			)
 		)
-		(property "Footprint" "NexusFC:F0805"
+		(property "Footprint" "NexusFC:F0805__NexusMain_F2"
 			(at 207.01 359.41 0)
 			(effects
@@
 			)
 		)
-		(property "Footprint" "NexusFC:CRYSTAL-SMD_4P-L3.2-W2.5-BL"
+		(property "Footprint" "NexusFC:CRYSTAL-SMD_4P-L3.2-W2.5-BL__NexusMain_Y1"
 			(at 341.63 229.87 0)
 			(effects
@@
 			)
 		)
-		(property "Footprint" "NexusFC:F0805"
+		(property "Footprint" "NexusFC:F0805__NexusMain_F1"
 			(at 728.98 76.2 0)
 			(effects
@@
 			)
 		)
-		(property "Footprint" "NexusFC:CONN-SMD_4P-P1.25_BM04B-GHS-TBT-LF-SN"
+		(property "Footprint" "NexusFC:CONN-SMD_4P-P1.25_BM04B-GHS-TBT-LF-SN__NexusMain_J3"
 			(at 590.55 196.85 90)
 			(effects
@@
 			)
 		)
-		(property "Footprint" "NexusFC:CONN-SMD_4P-P1.25_BM04B-GHS-TBT-LF-SN"
+		(property "Footprint" "NexusFC:CONN-SMD_4P-P1.25_BM04B-GHS-TBT-LF-SN__NexusMain_J5"
 			(at 782.32 196.85 90)
 			(effects
@@
 			)
 		)
-		(property "Footprint" "NexusFC:CONN-SMD_B3B-ZR-SM4-TF"
+		(property "Footprint" "NexusFC:CONN-SMD_B3B-ZR-SM4-TF__NexusMain_J2"
 			(at 788.67 265.43 0)
 			(effects
@@
 			)
 		)
-		(property "Footprint" "Resistor_SMD:R_0402_1005Metric"
+		(property "Footprint" "NexusFC:R_0402_1005Metric__NexusMain_R2"
 			(at 585.47 521.97 90)
 			(effects
@@
 			)
 		)
-		(property "Footprint" "Resistor_SMD:R_0402_1005Metric"
+		(property "Footprint" "NexusFC:R_0402_1005Metric__NexusMain_R4"
 			(at 759.46 521.97 90)
 			(effects

Commit message: tidy up traces
Parts:
- F1: footprint NexusFC:F0805__NexusMain_F1 -> NexusFC:F0805
- F2: footprint NexusFC:F0805__NexusMain_F2 -> NexusFC:F0805
- J2: footprint NexusFC:CONN-SMD_B3B-ZR-SM4-TF__NexusMain_J2 -> NexusFC:CONN-SMD_B3B-ZR-SM4-TF
- J3: footprint NexusFC:CONN-SMD_4P-P1.25_BM04B-GHS-TBT-LF-SN__NexusMain_J3 -> NexusFC:CONN-SMD_4P-P1.25_BM04B-GHS-TBT-LF-SN
- J5: footprint NexusFC:CONN-SMD_4P-P1.25_BM04B-GHS-TBT-LF-SN__NexusMain_J5 -> NexusFC:CONN-SMD_4P-P1.25_BM04B-GHS-TBT-LF-SN
- L2: footprint NexusFC:IND-SMD_L2.0-W1.6__NexusMain_L2 -> NexusFC:IND-SMD_L2.0-W1.6
- R2: footprint NexusFC:R_0402_1005Metric__NexusMain_R2 -> Resistor_SMD:R_0402_1005Metric
- R4: footprint NexusFC:R_0402_1005Metric__NexusMain_R4 -> Resistor_SMD:R_0402_1005Metric
- Y1: footprint NexusFC:CRYSTAL-SMD_4P-L3.2-W2.5-BL__NexusMain_Y1 -> NexusFC:CRYSTAL-SMD_4P-L3.2-W2.5-BL
Other:
- moved on the sheet: U11

Commit message: updated bom
Parts:
- added R23: 0.12, NexusFC:R_0402_1005Metric__VCAP_Dense, symbol Device:R
- C9: footprint Capacitor_SMD:C_0603_1608Metric -> NexusFC:C_0402_1005Metric__VCAP_Dense; LCSC C69335 -> C368809
- D4: value SMF13A -> SMF9.0A; footprint NexusFC:SOD-123FL_L2.8-W1.8-LS3.6-RD -> NexusFC:SOD-123FL_L2.8-W1.8-LS3.6-RD__Littelfuse_SMF9; symbol NexusFC:SMF13A_C353315 -> NexusReviewed:SMF9_0A_C1973343; LCSC C353315 -> C1973343
- F1: footprint NexusFC:F0805 -> NexusFC:F0805__NexusMain_F1
- F2: footprint NexusFC:F0805 -> NexusFC:F0805__NexusMain_F2
- J2: footprint NexusFC:CONN-SMD_B3B-ZR-SM4-TF -> NexusFC:CONN-SMD_B3B-ZR-SM4-TF__NexusMain_J2
- J3: footprint NexusFC:CONN-SMD_4P-P1.25_BM04B-GHS-TBT-LF-SN -> NexusFC:CONN-SMD_4P-P1.25_BM04B-GHS-TBT-LF-SN__NexusMain_J3
- J5: footprint NexusFC:CONN-SMD_4P-P1.25_BM04B-GHS-TBT-LF-SN -> NexusFC:CONN-SMD_4P-P1.25_BM04B-GHS-TBT-LF-SN__NexusMain_J5
- L2: footprint NexusFC:IND-SMD_L2.0-W1.6 -> NexusFC:IND-SMD_L2.0-W1.6__NexusMain_L2
- R2: footprint Resistor_SMD:R_0402_1005Metric -> NexusFC:R_0402_1005Metric__NexusMain_R2
- R4: footprint Resistor_SMD:R_0402_1005Metric -> NexusFC:R_0402_1005Metric__NexusMain_R4
- Y1: footprint NexusFC:CRYSTAL-SMD_4P-L3.2-W2.5-BL -> NexusFC:CRYSTAL-SMD_4P-L3.2-W2.5-BL__NexusMain_Y1
Connections:
- net VCAP: now also R23.1; no longer C9.1
- new net VCAP_C: C9.1, R23.2
