File: nexus-style-fc/routing-wip/current/hardware/nexus-style-fc.kicad_sch (KiCad schematic)
At the start: 88 parts, among them J1 Header child board, J2 DSM (UART1), J3 A-CRSF (UART4), J4 C (UART3), J5 B (UART6), J6 USB-C vertical, SW1 BOOT, U1 STM32F722RET6, U10 TPS70933DBVR, U11 SRV05-4, U12 SRV05-4, U13 SRV05-4, U14 TPS629210DRLR, U15 SRV05-4, U2 ICM-42688-P, U3 DPS368XTSA1, U4 W25N01GVZEIG, U5 TPS62130RGTR, U7 USBLC6-2SC6, U9 TPS2116DRLR, Y1 8MHz 20pF

Commit message: Nexus WIP: publish r62 input-cap star with zero native errors
Parts:
- added C31: 22uF, NexusFC:C_0805_2012Metric_Samsung_CL21_MinLand, symbol Device:C
- C27: value 4.7uF -> 22uF; footprint Capacitor_SMD:C_0603_1608Metric -> NexusFC:C_0805_2012Metric_Samsung_CL21_MinLand; LCSC C69335 -> C602037
Connections:
- net GND: now also C31.2
- net VSYS: now also C31.1
Changed lines of the file:
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@@
 			)
 		)
-		(property "Value" "4.7uF"
+		(property "Value" "22uF"
 			(at 102.87 328.93 0)
 			(effects
@@
 			)
 		)
-		(property "Footprint" "Capacitor_SMD:C_0603_1608Metric"
+		(property "Footprint" "NexusFC:C_0805_2012Metric_Samsung_CL21_MinLand"
 			(at 99.06 327.66 0)
 			(effects
@@
 			)
 		)
-		(property "LCSC" "C69335"
-			(at 99.06 327.66 0)
-			(effects
-				(font
-					(size 1.27 1.27)
-				)
-				(hide yes)
-			)
-		)
-		(property "Description" "buck in, 25 V"
+		(property "LCSC" "C602037"
+			(at 99.06 327.66 0)
+			(effects
+				(font
+					(size 1.27 1.27)
+				)
+				(hide yes)
+			)
+		)
+		(property "Description" "Main VSYS input bulk; Samsung CL21A226MAYNNNE; 22 uF, 25 V, X5R, +/-20%; JLC/LCSC C602037"
 			(at 99.06 327.66 0)
 			(effects
@@
 		)
 	)
+	(symbol
+		(lib_id "Device:C")
+		(at 71.12 327.66 0)
+		(unit 1)
+		(exclude_from_sim no)
+		(in_bom yes)
+		(on_board yes)
+		(dnp no)
+		(property "Reference" "C31"
+			(at 74.93 326.39 0)
+			(effects
+				(font
+					(size 1.27 1.27)
+				)
+				(justify left)
+			)
+		)
+		(property "Value" "22uF"
+			(at 74.93 328.93 0)
+			(effects
+				(font
+					(size 1.27 1.27)
+				)
+				(justify left)
+			)
+		)
+		(property "Footprint" "NexusFC:C_0805_2012Metric_Samsung_CL21_MinLand"
+			(at 71.12 327.66 0)
+			(effects
+				(font
+					(size 1.27 1.27)
+				)
+				(hide yes)
+			)
+		)
+		(property "Datasheet" ""
+			(at 71.12 327.66 0)
+			(effects
+				(font
+					(size 1.27 1.27)
+				)
+				(hide yes)
+			)
+		)
+		(property "LCSC" "C602037"
+			(at 71.12 327.66 0)
+			(effects
+				(font
+					(size 1.27 1.27)
+				)
+				(hide yes)
+			)
+		)
+		(property "Description" "Main VSYS local parallel input bulk; Samsung CL21A226MAYNNNE; 22 uF, 25 V, X5R, +/-20%; JLC/LCSC C602037"
+			(at 71.12 327.66 0)
+			(effects
+				(font
+					(size 1.27 1.27)
+				)
+				(hide yes)
+			)
+		)
+		(pin "1"
+		)
+		(pin "2"
+		)
+		(instances
+			(project "nexus-style-fc"
+				(path "/b1e839ec-d91a-58d5-9282-f5372deabfab"
+					(reference "C31")
+					(unit 1)
+				)
+			)
+		)
+	)
+	(wire
+		(pts
+			(xy 71.12 323.85)
+			(xy 71.12 317.5)
+		)
+		(stroke
+			(width 0)
+			(type default)
+		)
+	)
+	(junction
+		(at 71.12 317.5)
+		(diameter 0)
+		(color 0 0 0 0)
+	)
+	(wire
+		(pts
+			(xy 71.12 331.47)
+			(xy 71.12 340.36)
+		)
+		(stroke
+			(width 0)
+			(type default)
+		)
+	)
+	(wire
+		(pts
+			(xy 71.12 340.36)
+			(xy 99.06 340.36)
+		)
+		(stroke
+			(width 0)
+			(type default)
+		)
+	)
+	(junction
+		(at 99.06 340.36)
+		(diameter 0)
+		(color 0 0 0 0)
+	)
 	(global_label "VSYS"

Commit message: Nexus WIP: source-consistent assembly markings and release-gate evidence
Parts:
- D1: footprint NexusFC:LED0603-RD_GREEN -> NexusFC:LED0603-RD_GREEN__NexusMain_D1
- D2: footprint NexusFC:LED0603-RD_RED -> NexusFC:LED0603-RD_RED__NexusMain_D2
- D3: footprint NexusFC:LED0603-RD_BLUE -> NexusFC:LED0603-RD_BLUE__NexusMain_D3
- J4: footprint NexusFC:CONN-SMD_4P-P1.25_BM04B-GHS-TBT-LF-SN -> NexusFC:CONN-SMD_4P-P1.25_BM04B-GHS-TBT-LF-SN__NexusMain_J4
- J6: footprint NexusFC:USB-C-SMD_TYPE-C-31-D-06 -> NexusFC:USB-C-SMD_TYPE-C-31-D-06__NexusMain_J6
Changed lines of the file:
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@@
 			)
 		)
-		(property "Footprint" "NexusFC:USB-C-SMD_TYPE-C-31-D-06"
+		(property "Footprint" "NexusFC:USB-C-SMD_TYPE-C-31-D-06__NexusMain_J6"
 			(at 608.33 96.52 0)
 			(effects
@@
 			)
 		)
-		(property "Footprint" "NexusFC:CONN-SMD_4P-P1.25_BM04B-GHS-TBT-LF-SN"
+		(property "Footprint" "NexusFC:CONN-SMD_4P-P1.25_BM04B-GHS-TBT-LF-SN__NexusMain_J4"
 			(at 590.55 265.43 90)
 			(effects
@@
 			)
 		)
-		(property "Footprint" "NexusFC:LED0603-RD_GREEN"
+		(property "Footprint" "NexusFC:LED0603-RD_GREEN__NexusMain_D1"
 			(at 612.14 524.51 0)
 			(effects
@@
 			)
 		)
-		(property "Footprint" "NexusFC:LED0603-RD_RED"
+		(property "Footprint" "NexusFC:LED0603-RD_RED__NexusMain_D2"
 			(at 698.5 524.51 0)
 			(effects
@@
 			)
 		)
-		(property "Footprint" "NexusFC:LED0603-RD_BLUE"
+		(property "Footprint" "NexusFC:LED0603-RD_BLUE__NexusMain_D3"
 			(at 786.13 524.51 0)
 			(effects
