File: nexus-style-fc/hardware/header-board/nexus-header-board.kicad_sch (KiCad schematic)
At the start: 12 parts, among them J1 Servo header 3x7, K1 GND strip, K2 VX strip, P1 S1 tab pad, P2 S2 tab pad, P3 S3 tab pad, P4 TAIL tab pad, P5 ESC tab pad, P6 RPM tab pad, P7 SBUS tab pad, T1 GND tab pad, T2 VX tab pad

Commit message: Consolidate Nexus stage36 into canonical project paths
Preserve matched native sources and manufacturing bytes; use Git history for older project snapshots. Retain revision-bound validation evidence, document open release gates, and guard destructive regeneration.
Parts:
- K1, K2: footprint NexusFC:ChildBoard_TabStrip_W9.8 -> NexusFC:ChildBoard_TabStrip_W7.892
Changed lines of the file:
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@@
 			)
 		)
-		(property "Footprint" "NexusFC:ChildBoard_TabStrip_W9.8"
+		(property "Footprint" "NexusFC:ChildBoard_TabStrip_W7.892"
 			(at 130.81 36.83 0)
 			(effects
@@
 			)
 		)
-		(property "Footprint" "NexusFC:ChildBoard_TabStrip_W9.8"
+		(property "Footprint" "NexusFC:ChildBoard_TabStrip_W7.892"
 			(at 158.75 36.83 0)
 			(effects

Commit message: fix(nexus): clean up native fabrication warnings and bind verified exports
Center existing via connections, fix mixed USB connector classification,
move conflicting outline artwork to Fab layers, and synchronize reviewed
symbol/footprint identities. Preserve accepted pads, pinouts and parts.

Regenerate main CAM and record full KiCad 10 ERC/DRC/parity and source/CAM
consistency evidence. Keep remaining factory and bench qualification gates
explicit; this checkpoint is not a fabrication or flight release.
Parts:
- K1, K2, P1, P2, P3, P4, P5, P6, P7, T1, T2: symbol Connector_Generic:Conn_01x01 -> NexusReviewed:ChildContact
Changed lines of the file:
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@@
 	)
 	(symbol
-		(lib_id "Connector_Generic:Conn_01x01")
+		(lib_id "NexusReviewed:ChildContact")
 		(at 73.66 36.83 0)
 		(unit 1)
@@
 	)
 	(symbol
-		(lib_id "Connector_Generic:Conn_01x01")
+		(lib_id "NexusReviewed:ChildContact")
 		(at 102.87 36.83 0)
 		(unit 1)
@@
 	)
 	(symbol
-		(lib_id "Connector_Generic:Conn_01x01")
+		(lib_id "NexusReviewed:ChildContact")
 		(at 130.81 36.83 0)
 		(unit 1)
@@
 	)
 	(symbol
-		(lib_id "Connector_Generic:Conn_01x01")
+		(lib_id "NexusReviewed:ChildContact")
 		(at 158.75 36.83 0)
 		(unit 1)
@@
 	)
 	(symbol
-		(lib_id "Connector_Generic:Conn_01x01")
+		(lib_id "NexusReviewed:ChildContact")
 		(at 186.69 36.83 0)
 		(unit 1)
@@
 	)
 	(symbol
-		(lib_id "Connector_Generic:Conn_01x01")
+		(lib_id "NexusReviewed:ChildContact")
 		(at 214.63 36.83 0)
 		(unit 1)
@@
 	)
 	(symbol
-		(lib_id "Connector_Generic:Conn_01x01")
+		(lib_id "NexusReviewed:ChildContact")
 		(at 241.3 36.83 0)
 		(unit 1)
@@
 	)
 	(symbol
-		(lib_id "Connector_Generic:Conn_01x01")
+		(lib_id "NexusReviewed:ChildContact")
 		(at 270.51 36.83 0)
 		(unit 1)
@@
 	)
 	(symbol
-		(lib_id "Connector_Generic:Conn_01x01")
+		(lib_id "NexusReviewed:ChildContact")
 		(at 300.99 36.83 0)
 		(unit 1)
@@
 	)
 	(symbol
-		(lib_id "Connector_Generic:Conn_01x01")
+		(lib_id "NexusReviewed:ChildContact")
 		(at 330.2 36.83 0)
 		(unit 1)
@@
 	)
 	(symbol
-		(lib_id "Connector_Generic:Conn_01x01")
+		(lib_id "NexusReviewed:ChildContact")
 		(at 360.68 36.83 0)
 		(unit 1)
